File: Hardware/Arduino-Pro-Mini_195x195inch_bike.sch (EAGLE design)
At the start: 31 parts, among them Q1 8/16/20MHz, U1 ATMEGA328, U2 MIC5205

Commit message: work update, bike draft
Parts:
- removed B1: MB1S, rectifier:MB1S
- added 1, 2, C5, C9: 100nF, SparkFun-Capacitors:2.2UF50V10%(1206)
- added 330UH1, 330UH2: DR125, inductors:DR125
- added 5V_OUT_ARK, GENERATOR_AC_EXTRA_1: (no value), con-ptr500:AK300/2
- added BATTERY_CHARGER_5V, K6: ZNS5106, relay:ZNS5106
- added BIKE, BIKE_EXTRA: MB1S, rectifier:MB1S
- added C4, C6, C7, C8: 220uF, SparkFun-Capacitors:100UF-63V-20%(ELECT)
- added D2, D4: 1N5819-B, diode:1N5819-B
- added IC1: XL6009_FROM_LM2596S, xl6009:XL6009_FROM_LM2596S
- added JP10, JP11, JP12, JP13, JP14, JP15: (no value), pinhead:PINHD-1X2
- added JP17: USB_, SparkFun-Connectors:USB_
- added JP4: USB_MICROB_PLUGCONN-11752, SparkFun-Connectors:USB_MICROB_PLUGCONN-11752
- added RX2, RX3: 330R, SparkFun-Passives:RESISTOR0805-RES
- added STEP-DOWN_X_TO_5V: LM2596S, national-semiconductor:LM2596S
- added UR2, UR3: 10k, rcl:R-TRIMM3296W
Connections:
- new net 3-4V_LI-ION: 2.1, 330UH2.1, C7.+, IC1.VIN, JP12.2
- new net 5V: 330UH1.2, BATTERY_CHARGER_5V2.O, C5.2, C6.+, JP10.2, JP4.VCC, K62.S, UR2.E
- new net 5V_FROM_BATTERY: C19.+, C8.+, C9.2, D4.C, JP14.2, JP15.2, K62.O, U2.EN, U2.IN, UR3.E
- new net BIKE: BIKE.AC2, GENERATOR_AC-1.KL
- new net BIKE+: 1.1, BIKE.+, BIKE_EXTRA.+, C4.+, STEP-DOWN_X_TO_5V.VIN
- new net N$15: C5.1, RX2.2, STEP-DOWN_X_TO_5V.FB, UR2.A, UR2.S
- new net N$16: BATTERY_CHARGER_5V2.P, JP13.2
- new net N$17: 330UH1.1, D2.C, STEP-DOWN_X_TO_5V.OUT
- new net N$19: IC1.FB, RX3.2, UR3.A, UR3.S
- new net N$21: 5V_OUT_ARK-2.KL, JP11.2, JP17.VBUS, K62.P
- new net N$25: K61.1
- new net N$26: BATTERY_CHARGER_5V1.1
- new net N$8: BIKE_EXTRA.AC2, GENERATOR_AC_EXTRA_1-1.KL
- new net N$9: BIKE_EXTRA.AC1, GENERATOR_AC_EXTRA_1-2.KL
- net GND: now also 1.2, 2.2, 5V_OUT_ARK-1.KL, BATTERY_CHARGER_5V1.2, BIKE.-, BIKE_EXTRA.-, C4.-, C6.-, C7.-, C8.-, C9.1, D2.A, IC1.GND, JP10.1, JP11.1, JP12.1, JP13.1, JP14.1, JP15.1, JP17.GND, JP4.GND, K61.2, RX2.1, RX3.1, STEP-DOWN_X_TO_5V.!ON!/OFF, STEP-DOWN_X_TO_5V.GND
- net N$5: now also 330UH2.2, D4.A, IC1.SW; no longer B1.AC2, GENERATOR_AC-1.KL
- net N$6: now also BIKE.AC1; no longer B1.AC1
- net RAW: no longer C19.+, U2.EN, U2.IN
Other:
- note added: "1GND 2 EN 3 SW 4 VIN 5 FB"
- note added: "INA219 pomiar pradu?"
- note added: "a moze arduino?"
- note added: "co gdy nie ma baterii"
- note added: "pomiar napiecia baterii"
- note added: "pomiar napiecia zasilania co x sekund"
- note added: "tu powinny byc wyprowadzenia dla wyswietlacza, dla licznika rowerowego, dla oswietlenia, dla buletooth"
- note added: "tutaj powinien byc modul baterii"
- note added: "zamiana na ssr?"
- moved on the sheet: GENERATOR_AC-1, GENERATOR_AC-2
