File: Hardware/Arduino-Pro-Mini_195x195inch_upsbike.brd (EAGLE design)
At the start: 99.8 x 99.8 mm, 65 parts, among them IC1 XL6009_FROM_LM2596S, K1 CQ1-12V, K2 JJM2W-12V, K3 ZNS5106, Q1 8/16/20MHz, U1 ATMEGA328, U2 MIC5205

Commit message: bikeups
Parts:
- added K4, K5, K6, K7: ZNS5106, relay:ZN5
Changed lines of the file:
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@@
 <attribute name="OC_FARNELL" value="unknown" x="-182.88" y="-189.23" size="1.778" layer="27" display="off"/>
+</element>
+<element name="K4" library="relay" package="ZN5" value="ZNS5106" x="-24.13" y="-109.22">
+<attribute name="OC_NEWARK" value="unknown" x="-24.13" y="-109.22" size="1.778" layer="27" display="off"/>
+<attribute name="MPN" value="" x="-24.13" y="-109.22" size="1.778" layer="27" display="off"/>
+<attribute name="MF" value="" x="-24.13" y="-109.22" size="1.778" layer="27" display="off"/>
+<attribute name="OC_FARNELL" value="unknown" x="-24.13" y="-109.22" size="1.778" layer="27" display="off"/>
+</element>
+<element name="K5" library="relay" package="ZN5" value="ZNS5106" x="-24.13" y="-125.73">
+<attribute name="OC_NEWARK" value="unknown" x="-24.13" y="-125.73" size="1.778" layer="27" display="off"/>
+<attribute name="MPN" value="" x="-24.13" y="-125.73" size="1.778" layer="27" display="off"/>
+<attribute name="MF" value="" x="-24.13" y="-125.73" size="1.778" layer="27" display="off"/>
+<attribute name="OC_FARNELL" value="unknown" x="-24.13" y="-125.73" size="1.778" layer="27" display="off"/>
+</element>
+<element name="K6" library="relay" package="ZN5" value="ZNS5106" x="-24.13" y="-142.24">
+<attribute name="OC_NEWARK" value="unknown" x="-24.13" y="-142.24" size="1.778" layer="27" display="off"/>
+<attribute name="MPN" value="" x="-24.13" y="-142.24" size="1.778" layer="27" display="off"/>
+<attribute name="MF" value="" x="-24.13" y="-142.24" size="1.778" layer="27" display="off"/>
+<attribute name="OC_FARNELL" value="unknown" x="-24.13" y="-142.24" size="1.778" layer="27" display="off"/>
+</element>
+<element name="K7" library="relay" package="ZN5" value="ZNS5106" x="-24.13" y="-158.75">
+<attribute name="OC_NEWARK" value="unknown" x="-24.13" y="-158.75" size="1.778" layer="27" display="off"/>
+<attribute name="MPN" value="" x="-24.13" y="-158.75" size="1.778" layer="27" display="off"/>
+<attribute name="MF" value="" x="-24.13" y="-158.75" size="1.778" layer="27" display="off"/>
+<attribute name="OC_FARNELL" value="unknown" x="-24.13" y="-158.75" size="1.778" layer="27" display="off"/>
 </element>
 </elements>

Commit message: some work, not ready
Parts:
- removed >5V_OUT: (no value), con-ptr500:AK300/2
- removed K3, K4, K7: ZNS5106, relay:ZN5
- removed L1, L2, L3: 330uH, SparkFun-Passives:INDUCTOR-SRP4020
- added 330UH, 330UH1, 330UH2: DR125, inductors:DR125
- added 5V_OUT, BATTERY_CHARGER_5V: ZNS5106, relay:ZN5
- added >14V_IN1, >14V_IN2: (no value), con-ptr500:AK300/2
- added JP10, JP11, JP12, JP13, JP14, JP15, JP16, JP9: (no value), pinhead:1X02
- moved UR3 186.9 mm to (82.5, 72.4), turned to 180 degrees
- moved D4 183.7 mm to (71.1, 63.5), turned to 180 degrees
- moved RX3 177.9 mm to (86.4, 73.7), turned to 90 degrees
- moved D2 176.3 mm to (39.4, 64.8), turned to 180 degrees
- moved UR2 175.5 mm to (52.1, 71.1), turned to 180 degrees
- moved 13 168.7 mm to (21.6, 72.4), turned to 90 degrees
- moved C5 168.4 mm to (55.9, 66.0), turned to 90 degrees
- moved 2 164.5 mm to (80.0, 47.0)
- moved 1 163.0 mm to (34.3, 62.2)
- moved RX2 162.0 mm to (52.1, 64.8)
- moved UR1 159.5 mm to (22.9, 62.2), turned to 180 degrees
- moved C14 156.5 mm to (26.7, 61.0), turned to 270 degrees
- moved RX1 156.3 mm to (29.2, 61.0), turned to 90 degrees
- moved C7 155.0 mm to (71.1, 41.9)
- moved C11 153.2 mm to (14.0, 76.2), turned to 270 degrees
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Connections:
- removed net N$10: 13.1, >14V_IN.1, C11.+, STEP-DOWN_X_TO_13,7.1
- new net N$11: BATTERY_CHARGER_5V.12, K6.12
- new net N$14: 5V_OUT.12, JP11.1, K6.11
- new net N$16: BATTERY_CHARGER_5V.11, JP13.2
- new net N$18: >14V_IN1.1, JP9.1, K5.12
- new net N$20: 13.1, >14V_IN.2, C11.+, STEP-DOWN_X_TO_13,7.1
- new net N$21: 5V_OUT.11, >14V_IN2.1, JP16.1
- new net N$23: K5.A1
- new net N$24: 5V_OUT.A1
- new net N$25: K6.A1
- new net N$26: BATTERY_CHARGER_5V.A1
- net 13,7: now also 330UH.2, K5.11; no longer L1.P$2
- net 3-4V_LI-ION: now also 330UH2.1, JP12.2; no longer L3.P$1
- net 5V: now also 330UH1.2, JP10.1; no longer L2.P$2
- net 5V_FROM_BATTERY: now also JP14.1, K6.14
- net GND: now also 5V_OUT.A2, >14V_IN.1, >14V_IN1.2, >14V_IN2.2, BATTERY_CHARGER_5V.A2, JP10.2, JP11.2, JP12.1, JP13.1, JP14.2, JP16.2, K5.A2, K6.A2; no longer >14V_IN.2, >5V_OUT.2
- net N$12: now also 330UH.1; no longer L1.P$1
- net N$17: now also 330UH1.1; no longer L2.P$1
- net N$19: now also UR3.2
- net N$5: now also 330UH2.2; no longer L3.P$2
- net RAW: now also JP15.1
Routing:
- net GND: track 9.36 -> 124.6 mm, vias 13 -> 16
- net 13,7: track 0.00 -> 66.5 mm, vias 0 -> 2
- net 5V_FROM_BATTERY: track 0.00 -> 61.6 mm
- net N$12: track 0.00 -> 40.6 mm
- net N$20: track 0.00 -> 39.8 mm, vias 0 -> 2
- net 3-4V_LI-ION: track 0.00 -> 38.6 mm
- net 5V: track 0.00 -> 31.5 mm
- net N$5: track 0.00 -> 23.9 mm, vias 0 -> 1
- net N$17: track 0.00 -> 22.6 mm
- net N$15: track 0.00 -> 19.6 mm
- net N$13: track 0.00 -> 15.0 mm
- net N$19: track 0.00 -> 12.5 mm
Other:
- outline, holes or cut-outs redrawn
- board text added: "13,7V"
- board text added: "5v"
- board text added: "5v_bat"

Commit message: before ground
Parts:
- removed >14V_IN1, >14V_IN2: (no value), con-ptr500:AK300/2
- removed X1: (no value), con-yamaichi:USB-A003
- added 5V_OUT_ARK, >13.7V_BAT: (no value), con-ptr500:AK300/2
- added JP17: USB_, SparkFun-Connectors:USB-A-S-SILK-FEMALE
- moved JP13 331.6 mm to (91.4, 41.9)
- moved BATTERY_CHARGER_5V 326.4 mm to (92.7, 55.9), turned to 270 degrees
- moved JP16 311.2 mm to (90.2, 14.0)
- moved 5V_OUT 285.4 mm to (92.7, 27.9), turned to 270 degrees
- moved JP12 257.3 mm to (80.0, 40.6), turned to 90 degrees
- moved JP15 238.7 mm to (21.6, 22.9), turned to 90 degrees
- moved JP11 222.1 mm to (62.2, 16.5)
- moved JP9 215.5 mm to (11.4, 39.4), turned to 90 degrees
- moved JP10 210.1 mm to (47.0, 16.5)
- moved K6 187.0 mm to (53.3, 27.9)
- moved K5 169.1 mm to (30.5, 34.3), turned to 180 degrees
- moved JP4 167.6 mm to (97.8, 73.7), turned to 180 degrees
- moved GENERATOR_AC 30.5 mm to (63.5, 6.35)
- moved 330UH 1.27 mm to (7.62, 50.8)
- turned JP14 to 0 degrees
Connections:
- removed net N$11: BATTERY_CHARGER_5V.12, K6.12
- net 5V: now also BATTERY_CHARGER_5V.12, JP10.2, JP4.VBUS1, K6.12; no longer JP10.1
- net 5V_FROM_BATTERY: now also JP14.2; no longer JP14.1
- net GND: now also 5V_OUT_ARK.1, >13.7V_BAT.1, JP10.1, JP11.1, JP14.1, JP15.1, JP16.1, JP17.GND, JP4.GND1, JP9.1; no longer >14V_IN1.2, >14V_IN2.2, JP10.2, JP11.2, JP14.2, JP16.2
- net N$14: now also JP11.2; no longer JP11.1
- net N$18: now also >13.7V_BAT.2, JP9.2; no longer >14V_IN1.1, JP9.1
- net N$21: now also 5V_OUT_ARK.2, JP16.2, JP17.VBUS; no longer >14V_IN2.1, JP16.1
- net RAW: now also JP15.2; no longer JP15.1
Routing:
- net GND: track 124.6 -> 433.6 mm, vias 16 -> 21
- net 5V: track 31.5 -> 110.8 mm, vias 0 -> 3
- net N$14: track 0.00 -> 41.8 mm
- net N$21: track 0.00 -> 39.3 mm
- net N$18: track 0.00 -> 36.6 mm
- net 5V_FROM_BATTERY: track 61.6 -> 91.8 mm, vias 0 -> 1
- net 13,7: track 66.5 -> 83.5 mm
- net RAW: track 14.1 -> 22.7 mm
- net N$16: track 0.00 -> 5.08 mm
- net 3-4V_LI-ION: track 38.6 -> 43.0 mm
- net N$49: track 0.00 -> 2.54 mm, vias 0 -> 1
- net N$12: track 40.6 -> 39.4 mm
Other:
- board size 99.8 x 99.8 mm -> 99.8 x 84.6 mm

Commit message: work update, bike draft
Parts:
- removed D1, D2, D4: 1N5819-B, diode:DO41-7.6
- added D5, D6, D7: (no value), SparkFun-DiscreteSemi:SMA-DIODE_ALT
- moved GENERATOR_AC 7.41 mm to (69.8, 2.54)
- turned 5V_OUT_ARK to 0 degrees
Connections:
- net 5V_FROM_BATTERY: now also D7.C; no longer D4.C
- net GND: now also D5.A, D6.A; no longer D1.A, D2.A
- net N$12: now also D6.C; no longer D1.C
- net N$17: now also D5.C; no longer D2.C
- net N$5: now also D7.A; no longer D4.A
Routing:
- net SCK: track 9.93 -> 123.4 mm, vias 0 -> 1
- net MOSI: track 17.1 -> 111.6 mm, vias 1 -> 3
- net MISO: track 19.7 -> 114.1 mm
- net N$14: track 41.8 -> 82.7 mm, vias 0 -> 1
- net GND: track 433.6 -> 451.3 mm, vias 21 -> 22
- net N$21: track 39.3 -> 31.1 mm
- net D10: track 25.4 -> 33.6 mm
- net 5V_FROM_BATTERY: track 91.8 -> 96.2 mm, vias 1 -> 2
- net N$12: track 39.4 -> 42.5 mm
- net N$5: track 23.9 -> 25.8 mm
- net N$17: track 22.6 -> 23.2 mm
Other:
- board text added: "13.7V"
- board text added: "5V_Bat"
- board text removed: "13,7V"
- board text removed: "5v"
- board text removed: "5v_bat"
