File: Hardware/Arduino-Pro-Mini_195x195inch_upsbike.sch (EAGLE design)
At the start: 65 parts, among them IC1 XL6009_FROM_LM2596S, K1 CQ1-12V, K2 JJM2W-12V, K3 ZNS5106, Q1 8/16/20MHz, U1 ATMEGA328, U2 MIC5205

Commit message: bikeups
Parts:
- added K4, K5, K6, K7: ZNS5106, relay:ZNS5106
Other:
- note added: "BATERIA"
- moved on the sheet: K1, K2, K3
Changed lines of the file:
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@@
 <part name="K2" library="relay" deviceset="JJM2W-12V" device=""/>
 <part name="K3" library="relay" deviceset="ZNS5*" device="" technology="106"/>
+<part name="K4" library="relay" deviceset="ZNS5*" device="" technology="106"/>
+<part name="K5" library="relay" deviceset="ZNS5*" device="" technology="106"/>
+<part name="K6" library="relay" deviceset="ZNS5*" device="" technology="106"/>
+<part name="K7" library="relay" deviceset="ZNS5*" device="" technology="106"/>
 </parts>
 <sheets>
@@
 <text x="-228.6" y="139.7" size="1.778" layer="91">a moze arduino?</text>
 <text x="-193.04" y="20.32" size="1.778" layer="91">a moze arduino?</text>
+<text x="-55.88" y="276.86" size="1.778" layer="91">BATERIA</text>
 </plain>
 <instances>
@@
 <instance part="GND10" gate="1" x="-223.52" y="7.62"/>
 <instance part="IC1" gate="G$1" x="-203.2" y="35.56"/>
-<instance part="K1" gate="1" x="-116.84" y="-15.24"/>
-<instance part="K1" gate="2" x="-99.06" y="-15.24"/>
-<instance part="K2" gate="1" x="-165.1" y="-12.7"/>
-<instance part="K2" gate="2" x="-147.32" y="-12.7"/>
-<instance part="K3" gate="1" x="-215.9" y="-10.16"/>
-<instance part="K3" gate="2" x="-198.12" y="-10.16"/>
+<instance part="K1" gate="1" x="-434.34" y="45.72"/>
+<instance part="K1" gate="2" x="-416.56" y="45.72"/>
+<instance part="K2" gate="1" x="-414.02" y="-2.54"/>
+<instance part="K2" gate="2" x="-401.32" y="0"/>
+<instance part="K3" gate="1" x="-292.1" y="45.72"/>
+<instance part="K3" gate="2" x="-294.64" y="25.4"/>
+<instance part="K4" gate="1" x="-96.52" y="208.28"/>
+<instance part="K4" gate="2" x="-78.74" y="210.82"/>
+<instance part="K5" gate="1" x="-93.98" y="276.86"/>
+<instance part="K5" gate="2" x="-73.66" y="276.86"/>
+<instance part="K6" gate="1" x="-48.26" y="104.14" rot="R90"/>
+<instance part="K6" gate="2" x="-45.72" y="124.46" rot="R90"/>
+<instance part="K7" gate="1" x="-73.66" y="50.8" rot="R90"/>
+<instance part="K7" gate="2" x="-71.12" y="71.12" rot="R90"/>
 </instances>
 <busses>

Commit message: some work, not ready
Parts:
- removed >5V_OUT: (no value), con-ptr500:AK300/2
- removed K3, K4, K7: ZNS5106, relay:ZNS5106
- removed L1, L2, L3: 330uH, SparkFun-Passives:INDUCTOR
- added 330UH, 330UH1, 330UH2: DR125, inductors:DR125
- added 5V_OUT, BATTERY_CHARGER_5V: ZNS5106, relay:ZNS5106
- added >14V_IN1, >14V_IN2: (no value), con-ptr500:AK300/2
- added JP10, JP11, JP12, JP13, JP14, JP15, JP16, JP9: (no value), pinhead:PINHD-1X2
Connections:
- removed net N$10: 13.1, >14V_IN-1.KL, C11.+, STEP-DOWN_X_TO_13,7.VIN
- new net N$11: BATTERY_CHARGER_5V2.O, K62.O
- new net N$14: 5V_OUT2.O, JP11.1, K62.P
- new net N$16: BATTERY_CHARGER_5V2.P, JP13.2
- new net N$18: >14V_IN1-1.KL, JP9.1, K52.O
- new net N$20: 13.1, >14V_IN-2.KL, C11.+, STEP-DOWN_X_TO_13,7.VIN
- new net N$21: 5V_OUT2.P, >14V_IN2-1.KL, JP16.1
- new net N$23: K51.1
- new net N$24: 5V_OUT1.1
- new net N$25: K61.1
- new net N$26: BATTERY_CHARGER_5V1.1
- net 13,7: now also 330UH.2, K52.P; no longer L1.2
- net 3-4V_LI-ION: now also 330UH2.1, JP12.2; no longer L3.1
- net 5V: now also 330UH1.2, JP10.1; no longer L2.2
- net 5V_FROM_BATTERY: now also JP14.1, K62.S
- net GND: now also 5V_OUT1.2, >14V_IN-1.KL, >14V_IN1-2.KL, >14V_IN2-2.KL, BATTERY_CHARGER_5V1.2, JP10.2, JP11.2, JP12.1, JP13.1, JP14.2, JP16.2, K51.2, K61.2; no longer >14V_IN-2.KL, >5V_OUT-2.KL
- net N$12: now also 330UH.1; no longer L1.1
- net N$17: now also 330UH1.1; no longer L2.1
- net N$19: now also UR3.S
- net N$5: now also 330UH2.2; no longer L3.2
- net RAW: now also JP15.1
Other:
- moved on the sheet: >14V_IN-1, >14V_IN-2, JP4, K5, K6, X1

Commit message: before ground
Parts:
- removed >14V_IN1, >14V_IN2: (no value), con-ptr500:AK300/2
- removed X1: (no value), con-yamaichi:USB-A003
- added 5V_OUT_ARK, >13.7V_BAT: (no value), con-ptr500:AK300/2
- added JP17: USB_, SparkFun-Connectors:USB_
Connections:
- removed net N$11: BATTERY_CHARGER_5V2.O, K62.O
- net 5V: now also BATTERY_CHARGER_5V2.O, JP10.2, JP4.VCC, K62.O; no longer JP10.1
- net 5V_FROM_BATTERY: now also JP14.2; no longer JP14.1
- net GND: now also 5V_OUT_ARK-1.KL, >13.7V_BAT-1.KL, JP10.1, JP11.1, JP14.1, JP15.1, JP16.1, JP17.GND, JP4.GND, JP9.1; no longer >14V_IN1-2.KL, >14V_IN2-2.KL, JP10.2, JP11.2, JP14.2, JP16.2
- net N$14: now also JP11.2; no longer JP11.1
- net N$18: now also >13.7V_BAT-2.KL, JP9.2; no longer >14V_IN1-1.KL, JP9.1
- net N$21: now also 5V_OUT_ARK-2.KL, JP16.2, JP17.VBUS; no longer >14V_IN2-1.KL, JP16.1
- net RAW: now also JP15.2; no longer JP15.1
Other:
- moved on the sheet: JP10, JP11, JP14, JP15, JP16, JP4, JP9

Commit message: work update, bike draft
Parts:
- removed D1, D2, D4: 1N5819-B, diode:1N5819-B
- added D5, D6, D7: (no value), SparkFun-DiscreteSemi:DIODESMA-ALT
Connections:
- net 5V_FROM_BATTERY: now also D7.C; no longer D4.C
- net GND: now also D5.A, D6.A; no longer D1.A, D2.A
- net N$12: now also D6.C; no longer D1.C
- net N$17: now also D5.C; no longer D2.C
- net N$5: now also D7.A; no longer D4.A
Changed lines of the file:
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@@
 <part name="13" library="SparkFun-Capacitors" deviceset="2.2UF50V10%(1206)" device="" value="100nF"/>
 <part name="C14" library="SparkFun-Capacitors" deviceset="2.2UF50V10%(1206)" device="" value="100nF"/>
-<part name="D1" library="diode" deviceset="1N581*" device="" technology="9-B"/>
 <part name="RX1" library="SparkFun-Passives" deviceset="RESISTOR" device="0805-RES" value="330R"/>
 <part name="UR1" library="rcl" deviceset="R-TRIMM" device="3296W" value="10k"/>
@@
 <part name="C4" library="SparkFun-Capacitors" deviceset="100UF-63V-20%(ELECT)" device="" value="220uF"/>
 <part name="RX2" library="SparkFun-Passives" deviceset="RESISTOR" device="0805-RES" value="330R"/>
-<part name="D2" library="diode" deviceset="1N581*" device="" technology="9-B"/>
 <part name="UR2" library="rcl" deviceset="R-TRIMM" device="3296W" value="10k"/>
 <part name="C5" library="SparkFun-Capacitors" deviceset="2.2UF50V10%(1206)" device="" value="100nF"/>
@@
 <part name="RX3" library="SparkFun-Passives" deviceset="RESISTOR" device="0805-RES" value="330R"/>
 <part name="UR3" library="rcl" deviceset="R-TRIMM" device="3296W" value="10k"/>
-<part name="D4" library="diode" deviceset="1N581*" device="" technology="9-B"/>
 <part name="GND10" library="SparkFun-Aesthetics" deviceset="GND" device=""/>
 <part name="IC1" library="xl6009" deviceset="XL6009_FROM_LM2596" device="S"/>
@@
 <part name="330UH2" library="inductors" deviceset="DR125" device=""/>
 <part name="JP17" library="SparkFun-Connectors" deviceset="USB" device="_"/>
+<part name="D5" library="SparkFun-DiscreteSemi" deviceset="DIODE" device="SMA-ALT"/>
+<part name="D6" library="SparkFun-DiscreteSemi" deviceset="DIODE" device="SMA-ALT"/>
+<part name="D7" library="SparkFun-DiscreteSemi" deviceset="DIODE" device="SMA-ALT"/>
 </parts>
 <sheets>
@@
 <instance part="13" gate="G$1" x="-238.76" y="213.36"/>
 <instance part="C14" gate="G$1" x="-157.48" y="248.92" rot="R90"/>
-<instance part="D1" gate="G$1" x="-170.18" y="205.74" rot="R90"/>
 <instance part="RX1" gate="G$1" x="-180.34" y="205.74" rot="R90"/>
 <instance part="UR1" gate="G$1" x="-157.48" y="236.22" rot="MR90"/>
@@
 <instance part="C4" gate="G$1" x="-256.54" y="132.08"/>
 <instance part="RX2" gate="G$1" x="-180.34" y="127" rot="R90"/>
-<instance part="D2" gate="G$1" x="-167.64" y="127" rot="R90"/>
 <instance part="UR2" gate="G$1" x="-154.94" y="160.02" rot="MR90"/>
 <instance part="C5" gate="G$1" x="-154.94" y="172.72" rot="R90"/>
@@
 <instance part="RX3" gate="G$1" x="-167.64" y="27.94" rot="R90"/>
 <instance part="UR3" gate="G$1" x="-167.64" y="53.34" rot="MR0"/>
-<instance part="D4" gate="G$1" x="-180.34" y="71.12"/>
 <instance part="GND10" gate="1" x="-223.52" y="7.62"/>
 <instance part="IC1" gate="G$1" x="-203.2" y="35.56"/>
@@
 <instance part="330UH2" gate="G$1" x="-218.44" y="71.12"/>
 <instance part="JP17" gate="G$1" x="12.7" y="213.36"/>
+<instance part="D5" gate="G$1" x="-167.64" y="127" rot="R90"/>
+<instance part="D6" gate="G$1" x="-170.18" y="205.74" rot="R90"/>
+<instance part="D7" gate="G$1" x="-180.34" y="71.12"/>
 </instances>
 <busses>
@@
 <wire x1="-218.44" y1="215.9" x2="-218.44" y2="210.82" width="0.1524" layer="91"/>
 <pinref part="RX1" gate="G$1" pin="1"/>
-<pinref part="D1" gate="G$1" pin="A"/>
 <wire x1="-129.54" y1="200.66" x2="-129.54" y2="190.5" width="0.1524" layer="91"/>
 <junction x="-129.54" y="190.5"/>
@@
 <wire x1="-284.48" y1="210.82" x2="-271.78" y2="210.82" width="0.4064" layer="91"/>
 <wire x1="-266.7" y1="210.82" x2="-271.78" y2="210.82" width="0.4064" layer="91"/>
+<pinref part="D6" gate="G$1" pin="A"/>
 </segment>
 <segment>
@@
 <pinref part="RX2" gate="G$1" pin="1"/>
 <junction x="-220.98" y="111.76"/>
-<pinref part="D2" gate="G$1" pin="A"/>
 <wire x1="-220.98" y1="111.76" x2="-180.34" y2="111.76" width="0.1524" layer="91"/>
 <wire x1="-180.34" y1="111.76" x2="-167.64" y2="111.76" width="0.1524" layer="91"/>
@@
 <pinref part="JP10" gate="G$1" pin="1"/>
 <wire x1="-83.82" y1="139.7" x2="-73.66" y2="139.7" width="0.1524" layer="91"/>
+<pinref part="D5" gate="G$1" pin="A"/>
 </segment>
 <segment>
@@
 <net name="N$12" class="0">
 <segment>
-<pinref part="D1" gate="G$1" pin="C"/>
 <wire x1="-170.18" y1="208.28" x2="-170.18" y2="218.44" width="0.1524" layer="91"/>
 <wire x1="-170.18" y1="218.44" x2="-162.56" y2="218.44" width="0.1524" layer="91"/>
@@
 <junction x="-170.18" y="218.44"/>
 <pinref part="330UH" gate="G$1" pin="1"/>
+<pinref part="D6" gate="G$1" pin="C"/>
 </segment>
 </net>
@@
 <net name="N$17" class="0">
 <segment>
-<pinref part="D2" gate="G$1" pin="C"/>
 <wire x1="-167.64" y1="129.54" x2="-167.64" y2="142.24" width="0.1524" layer="91"/>
 <pinref part="STEP-DOWN_X_TO_5V" gate="G$1" pin="OUT"/>
@@
 <junction x="-167.64" y="142.24"/>
 <pinref part="330UH1" gate="G$1" pin="1"/>
+<pinref part="D5" gate="G$1" pin="C"/>
 </segment>
 </net>
@@
 <net name="N$5" class="0">
 <segment>
-<pinref part="D4" gate="G$1" pin="A"/>
 <wire x1="-210.82" y1="71.12" x2="-200.66" y2="71.12" width="0.1524" layer="91"/>
 <wire x1="-200.66" y1="71.12" x2="-182.88" y2="71.12" width="0.1524" layer="91"/>
@@
 <pinref part="IC1" gate="G$1" pin="SW"/>
 <pinref part="330UH2" gate="G$1" pin="2"/>
+<pinref part="D7" gate="G$1" pin="A"/>
 </segment>
 </net>
 <net name="5V_FROM_BATTERY" class="0">
 <segment>
-<pinref part="D4" gate="G$1" pin="C"/>
 <pinref part="UR3" gate="G$1" pin="E"/>
 <wire x1="-177.8" y1="71.12" x2="-167.64" y2="71.12" width="0.1524" layer="91"/>
@@
 <pinref part="JP14" gate="G$1" pin="2"/>
 <wire x1="-104.14" y1="50.8" x2="-86.36" y2="50.8" width="0.1524" layer="91"/>
-</segment>
-</net>
+<pinref part="D7" gate="G$1" pin="C"/>
+</segment>
+</net>
